Commit message: Added colors to links + Adjusted Camera Position

File: ohm_description/urdf/ohm.urdf (robot description, URDF)
Before this commit: robot ohm, 12 links, 11 joints
Joints:
- joint Camera_Link_to_base_link: origin xyz=0.2468 0 1.3716 rpy=0 0.785398 0 -> xyz=0.3992 0 1.3716 rpy=0 0.785398 0

Commit message: Created basic course / gazebo path adjustments

File: ohm_description/urdf/ohm.urdf (robot description, URDF)
Before this commit: robot ohm, 12 links, 11 joints
Joints:
- joint base_footprint_to_base_link: origin xyz=0 0 0 rpy=0 0 0 -> xyz=0 0 0.225 rpy=0 0 0
